Commit message: new 3dof arm

File: arm_description/urdf/arm_description.urdf (robot description, URDF)
Before this commit: robot arm_description, 3 links, 2 joints
Links:
- removed link Base_Link
- removed link Link_00
- removed link Link_01
- added link base_link, mass 0.51132; collision mesh filename=package://arm_description/meshes/base_link.STL; visual mesh filename=package://arm_description/meshes/base_link.STL
- added link link_00, mass 0.91073; collision mesh filename=package://arm_description/meshes/link_00.STL; visual mesh filename=package://arm_description/meshes/link_00.STL
- added link link_01, mass 1.0247; collision mesh filename=package://arm_description/meshes/link_01.STL; visual mesh filename=package://arm_description/meshes/link_01.STL
- added link link_02, mass 0.49537; collision mesh filename=package://arm_description/meshes/link_02.STL; visual mesh filename=package://arm_description/meshes/link_02.STL
Joints:
- removed joint Base_to_00
- added joint 01_to_02: type continuous, parent link_01, child link_02, origin xyz=0 0.15 0 rpy=-1.7159 -9.3328E-16 3.1416, axis 1 0 0
- added joint base_to_00: type continuous, parent base_link, child link_00, origin xyz=0 0 0.035 rpy=1.5708 -6.1219E-17 -1.5519, axis 0 1 0
- joint 00_to_01: axis 1 0 0 -> -1 0 0; child Link_01 -> link_01; origin xyz=0 0.07 0.078535 rpy=3.1384 -1.5708 0 -> xyz=0 0.07 0.080036 rpy=2.4677 -1.5708 0; parent Link_00 -> link_00

Commit message: fix urdf

File: arm_description/urdf/arm_description.urdf (robot description, URDF)
Before this commit: robot arm_model, 4 links, 3 joints
Links:
- added link world
- link base_link: mass 100.0 -> 0.511320
Joints:
- added joint world_joint: type fixed, parent world, child link_00

Commit message: added verbose

File: arm_description/urdf/arm_description.urdf (robot description, URDF)
Before this commit: robot arm_model, 5 links, 4 joints
Joints:
- joint 01_to_02: type continuous -> revolute

Commit message: one more try

File: arm_description/urdf/arm_description.urdf (robot description, URDF)
Before this commit: robot arm_model, 5 links, 4 joints
Joints:
- joint 01_to_02: limit lower=2 upper=3 effort=10 velocity=10 -> lower=-1 upper=0 effort=10 velocity=10

Commit message: joint changed to continuous

File: arm_description/urdf/arm_description.urdf (robot description, URDF)
Before this commit: robot arm_model, 5 links, 4 joints
Joints:
- joint 00_to_01: limit lower=2 upper=3 effort=10 velocity=10 -> effort=10 velocity=10; type revolute -> continuous
- joint 01_to_02: limit lower=-1 upper=0 effort=10 velocity=10 -> effort=10 velocity=10; type revolute -> continuous
